File: PCB/36mm PCB/_autosave-36mm PCB.kicad_pcb (KiCad board)
At the start: 2 copper layers, 29.3 x 14.5 mm, 64 parts, among them IC1 PCF2003DUS, IC2 BMM350, IC3 STM32L011E4Y6TR, IC4 TPS22991BRAAR, IC5 MCP73831-2ACI_MC, IC6 AS5510-DWLM, Q3 2N7002KQBZ, Q4 2N7002KQBZ, Q5 2N7002KQBZ, Q6 2N7002KQBZ, Q7 2N7002KQBZ, SW5 SW_MEC_5E, U1 BMP581, Y1 ABS04W-32.768KHZ-4-D2-T5

Commit message: PCB 2.0
Parts:
- removed C1, C13, C16, C4, C5: 100n, Capacitor_SMD:C_0201_0603Metric
- removed C12: 220n, Capacitor_SMD:C_0201_0603Metric
- removed C14: 4.7u, Capacitor_SMD:C_0201_0603Metric
- removed C2, C3, C6, C7: 1u, Capacitor_SMD:C_0201_0603Metric
- removed C8: 200n, Capacitor_SMD:C_0201_0603Metric
- removed D1, D2: D, Diode_SMD:D_0201_0603Metric
- removed IC3: STM32L011E4Y6TR, SamacSys_Parts:BGA25C40P5X5_213X207X58
- removed IC4: TPS22991BRAAR, SamacSys_Parts:TPS22991BRAAR
- removed IC6: AS5510-DWLM, SamacSys_Parts:BGA6C40P3X2_138X102X63
- removed L1: 27n, Inductor_SMD:L_0201_0603Metric
- removed R10: 100k, Resistor_SMD:R_0201_0603Metric
- removed TP1: GND_PCF2003, TestPoint:TestPoint_Pad_D1.0mm
- removed TP14: B+, TestPoint:TestPoint_Pad_D1.0mm
- removed TP15: B-, TestPoint:TestPoint_Pad_D1.0mm
- removed TP2: VDD_PCF2003, TestPoint:TestPoint_Pad_D1.0mm
- removed TP5: SWDIO, TestPoint:TestPoint_Pad_D1.0mm
- removed TP6: SWCLK, TestPoint:TestPoint_Pad_D1.0mm
- removed TP7: NRST, TestPoint:TestPoint_Pad_D1.0mm
- removed TPS3424-1: ~, Package_TO_SOT_SMD:SOT-583-8
- added C17: 100n, Capacitor_SMD:C_0201_0603Metric, F.Cu at (211.3, 118.3)
- added C18: 2.2u, Capacitor_SMD:C_0402_1005Metric, F.Cu at (207.6, 123.8)
- added C20: 220n, Capacitor_SMD:C_0201_0603Metric, F.Cu at (187.6, 118.5)
- added C21: 100n, Capacitor_SMD:C_0201_0603Metric, F.Cu at (189.9, 118.7)
- added C22: 4.7u, Capacitor_SMD:C_0402_1005Metric, F.Cu at (193.9, 123.7)
- added C23: 1u, Capacitor_SMD:C_0402_1005Metric, B.Cu at (196.7, 125.1)
- added C24: 100n, Capacitor_SMD:C_0201_0603Metric, B.Cu at (197.7, 125.0)
- added C25: 1u, Capacitor_SMD:C_0402_1005Metric, B.Cu at (194.7, 117.7)
- added C26: 1u, Capacitor_SMD:C_0402_1005Metric, F.Cu at (206.1, 121.2)
- added C27: 100n, Capacitor_SMD:C_0201_0603Metric, B.Cu at (204.1, 124.7)
- added C28: 100n, Capacitor_SMD:C_0201_0603Metric, B.Cu at (201.0, 126.9)
- added C29: 100n, Capacitor_SMD:C_0201_0603Metric, B.Cu at (202.9, 124.4)
- added C30: 1u, Capacitor_SMD:C_0402_1005Metric, B.Cu at (202.7, 125.3)
- added J1: Conn_01x04_Pin, SamacSys_Parts:Hall effect, F.Cu at (209.8, 116.4)
- added J2: Conn_01x02_Socket, SamacSys_Parts:Battery 36mm watch, F.Cu at (190.5, 115.3)
- added J3: Conn_01x02, SamacSys_Parts:Battery pogo pins, F.Cu at (193.3, 121.6)
- added LDLN025PU1: ~, Package_DFN_QFN:OnSemi_XDFN4-1EP_1.0x1.0mm_EP0.52x0.52mm, F.Cu at (193.8, 117.3)
- added LED1: 150060WS75000, SamacSys_Parts:150060WS75000, B.Cu at (192.9, 121.5)
- added R11: 10, Resistor_SMD:R_0402_1005Metric, B.Cu at (195.8, 117.7)
- added R20: 100k, Resistor_SMD:R_0201_0603Metric, B.Cu at (202.5, 126.2)
- added R22: 4.7k, Resistor_SMD:R_0201_0603Metric, B.Cu at (207.2, 118.1)
- added R23: 4.7k, Resistor_SMD:R_0201_0603Metric, B.Cu at (208.2, 118.1)
- added TP16: VDD Prog, SamacSys_Parts:Pogo pin 1x1, B.Cu at (204.4, 120.7)
- added TP19: NRST, SamacSys_Parts:Pogo pin 1x1, B.Cu at (204.1, 123.4)
- added TP20: 3.3V, SamacSys_Parts:Pogo pin 1x1, B.Cu at (195.7, 124.6)
- added TP21: VSS, SamacSys_Parts:Pogo pin 1x1, B.Cu at (197.5, 126.7)
- added TPS3424A11C13ADRLR1: ~, Package_TO_SOT_SMD:SOT-583-8, F.Cu at (191.5, 117.7)
- added U2: STM32L011F4Ux, Package_DFN_QFN:ST_UFQFPN-20_3x3mm_P0.5mm, B.Cu at (200.0, 124.7)
- C10, L2, L3, R19, SW5, U1: moved to B.Cu
- C15: footprint Capacitor_SMD:C_0201_0603Metric -> Capacitor_SMD:C_0402_1005Metric
- CLPT1: value 1u -> 11.8n; footprint Capacitor_SMD:C_0201_0603Metric -> Capacitor_SMD:C_0402_1005Metric
- CSPT1: value 1u -> 4.7n; footprint Capacitor_SMD:C_0201_0603Metric -> Capacitor_SMD:C_0402_1005Metric
- R15: value 100k -> 47k
- R16: value 100k -> 1k
- R17: value 1k -> 2k
- R18: value 47k -> 100k
- R3: value 0 -> 4.7k
- R4: value 2k -> 4.7k
- R5: value 2k -> 4.7k; moved to B.Cu
- R6: value 2k -> 500; moved to B.Cu
- R7, R8: value 2k -> 100k
- R9: value 0 -> 4.7k; moved to B.Cu
- TP17: value Charge+ -> SWDIO; footprint TestPoint:TestPoint_Pad_D1.0mm -> SamacSys_Parts:Pogo pin 1x1; moved to B.Cu
- TP18: value Charge- -> SWCLK; footprint TestPoint:TestPoint_Pad_D1.0mm -> SamacSys_Parts:Pogo pin 1x1; moved to B.Cu
- Y1: value ABS04W-32.768KHZ-4-D2-T5 -> LFXTAL062558Reel; footprint SamacSys_Parts:ABS04W32768KHZ4D2T5 -> SamacSys_Parts:LFXTAL062558Reel
- moved R17 98.6 mm to (199.1, 121.0), turned to -65 degrees
- moved CLPT1 97.2 mm to (193.2, 119.5), turned to 115 degrees
- moved R18 95.2 mm to (195.9, 121.1), turned to -65 degrees
- moved CSPT1 95.0 mm to (191.7, 120.2), turned to 115 degrees
- moved R19 95.0 mm to (204.0, 126.2), turned to 180 degrees
- moved C11 93.7 mm to (206.7, 124.0), turned to 90 degrees
- moved C9 92.7 mm to (205.8, 122.2), turned to 180 degrees
- moved R4 89.1 mm to (203.9, 122.9), turned to -90 degrees
- moved IC2 88.1 mm to (205.4, 123.5), turned to 90 degrees
- moved Y1 86.1 mm to (207.1, 118.3), turned to 90 degrees
- moved Q7 85.8 mm to (197.2, 120.4), turned to -65 degrees
- moved TP18 85.5 mm to (199.5, 121.8), turned to 180 degrees
- moved C15 84.6 mm to (194.8, 125.5), turned to -65 degrees
- moved TP17 83.7 mm to (197.2, 122.8), turned to 180 degrees
- moved R3 83.2 mm to (203.9, 124.4), turned to 90 degrees
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Connections:
- net Net-(IC1-VDD) renamed /Main dial/VDD PROG
- C10 pad 2: Net-(U1-VDDIO) -> /Peripherals/VDDIO
- C11 pad 2: Controller Output -> +3.3V
- C9 pad 1: Controller Output -> GND
- C9 pad 2: GND -> +3.3V
- IC1 pad B2: OSCIN -> /Main dial/OSCIN
- IC1 pad C1: OSCOUT -> /Main dial/OSCOUT
- IC2 pad A2: I2C1_SDA -> /I2C_SDA
- IC2 pad A3: I2C1_SCL -> /I2C_SCL
- IC2 pad B3: Controller Output -> +3.3V
- IC2 pad C1: Controller Output -> +3.3V
- IC5 pad 1: Charge+ -> /Power/Charge +
- IC5 pad 2: Charge+ -> /Power/Charge +
- IC5 pad 5: Stat -> /Power/STAT
- Q3 pad 1: Tim2_CH3 -> /H_Tim1
- Q3 pad 2: Controller Output -> +3.3V
- Q4 pad 1: Tim2_CH1 -> /H_Tim2
- Q4 pad 2: Controller Output -> +3.3V
- Q5 pad 1: Tim2_CH1 -> /H_Tim2
- Q6 pad 1: Tim2_CH3 -> /H_Tim1
- Q7 pad 1: Charge+ -> /Power/Charge +
- R13 pad 1: Controller Output -> Net-(Q4-D_1)
- R13 pad 2: Tim2_CH3 -> /H_Tim1
- R14 pad 1: Tim2_CH1 -> +3.3V
- R14 pad 2: Controller Output -> /H_Tim2
- R15 pad 1: Tim2_CH1 -> Net-(C20-Pad2)
- R15 pad 2: Net-(Q3-D_1) -> /Button press
- R16 pad 1: Net-(Q4-D_1) -> Net-(C20-Pad2)
- R16 pad 2: Tim2_CH3 -> GND
- R17 pad 1: GND -> Net-(Q7-D_1)
- R17 pad 2: Net-(C12-Pad2) -> Net-(IC5-PROG)
- R18 pad 1: Net-(C12-Pad2) -> /Power/Charge +
- R18 pad 2: GPIO_EXTI9 -> GND
- R19 pad 1: GND -> +3V0
- R19 pad 2: Charge+ -> Net-(U2-PA0)
- R3 pad 1: Net-(IC1-RESET) -> +3.3V
- R3 pad 2: +3V0 -> /I2C_SDA
- R4 pad 1: Controller Output -> +3.3V
- R4 pad 2: I2C1_SDA -> /I2C_SCL
- R5 pad 1: Controller Output -> /I2C_SCL
- R5 pad 2: I2C1_SCL -> +3.3V
- R6 pad 1: Net-(IC5-PROG) -> /Power/STAT
- R6 pad 2: Net-(Q7-D_1) -> Net-(LED1-K)
- R7 pad 1: I2C1_SCL -> +3.3V
- R7 pad 2: Controller Output -> /H_Tim1
- R8 pad 1: I2C1_SDA -> Net-(Q3-D_1)
- R8 pad 2: Controller Output -> /H_Tim2
- R9 pad 1: Controller Output -> +3.3V
- R9 pad 2: GND -> /I2C_SDA
- SW5 pad 1: Net-(C12-Pad2) -> Net-(C20-Pad2)
- SW5 pad 2: Net-(C12-Pad2) -> +3V0
- SW5 pad 3: +3V0 -> Net-(C20-Pad2)
- TP17 pad 1: Charge+ -> /SWDIO
- TP18 pad 1: GND -> /SWCLK
- U1 pad 1: Net-(U1-VDDIO) -> /Peripherals/VDDIO
- U1 pad 10: Controller Output -> /Peripherals/VDDIO
- U1 pad 2: I2C1_SCL -> /I2C_SCL
- U1 pad 4: I2C1_SDA -> /I2C_SDA
- U1 pad 6: unconnected-(U1-CSB-Pad6) -> /Peripherals/VDDIO
- U1 pad 7: GND -> /BMP581_INT
- Y1 pad 1: OSCIN -> /Main dial/OSCOUT
- Y1 pad 2: GND -> /Main dial/OSCIN
Routing:
- net /I2C_SDA: track 0.00 -> 33.7 mm, vias 0 -> 4
- net /I2C_SCL: track 0.00 -> 32.7 mm, vias 0 -> 4
- net +3.3V: track 0.00 -> 25.6 mm, vias 0 -> 15
- net /H_Tim1: track 0.00 -> 24.7 mm, vias 0 -> 2
- net /H_Tim2: track 0.00 -> 19.2 mm, vias 0 -> 2
- net /KeepOn: track 0.00 -> 17.4 mm, vias 0 -> 1
- net /Button press: track 0.00 -> 16.2 mm, vias 0 -> 1
- net /Kill: track 0.00 -> 14.9 mm, vias 0 -> 1
- net /BMP581_INT: track 0.00 -> 13.6 mm
- net /L-S press INT: track 0.00 -> 13.4 mm, vias 0 -> 1
- net /Main dial/VDD PROG: track 0.00 -> 6.17 mm, vias 0 -> 1
- net Net-(Q4-D_1): track 0.00 -> 6.02 mm, vias 0 -> 1
- net /Peripherals/VDDIO: track 0.00 -> 5.62 mm
- net Net-(IC1-RESET): track 0.00 -> 5.47 mm
- net /Power/STAT: track 0.00 -> 5.06 mm, vias 0 -> 1
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- added copper zone on F.Cu, net +3.3V
- added copper zone on In3.Cu, net +3.3V
- added copper zone on F.Cu, net +3V0
- added copper zone on In2.Cu, net +3V0
- added copper zone on F.Cu, net /Power/Charge +
- added copper zone on B.Cu, net GND
- added copper zone on F.Cu, net GND
- added copper zone on In1.Cu, net GND
- added copper zone on In4.Cu, net GND
- added copper zone on F.Cu, net Net-(C20-Pad2)
Other:
- board size 29.3 x 14.5 mm -> 29.1 x 14.4 mm
- copper layers 2 -> 6
