File: PCB/36mm PCB/MainDial.kicad_sch (KiCad schematic)
At the start: 6 parts, among them IC1 PCF2003DUS, Y1 LFXTAL062558Reel

Commit message: Modifs Mathieu
Parts:
- added R30: 0, Resistor_SMD:R_0201_0603Metric, symbol Device:R
Connections:
- net at IC1.A5 (RESET), R2.2: now also R30.1
- new net PCF_Reset: R30.2
Changed lines of the file:
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@@
+	)
+	(junction
+		(at 107.95 63.5)
+		(diameter 0)
+		(color 0 0 0 0)
 	)
 	(junction
@@
 			)
 			(justify right bottom)
+		)
+	)
+	(hierarchical_label "PCF_Reset"
+		(shape input)
+		(at 107.95 71.12 0)
+		(effects
+			(font
+				(size 1.27 1.27)
+			)
+			(justify left)
 		)
 	)
@@
 					(unit 1)
 				)
+			)
+		)
+	)
+	(symbol
+		(lib_id "Device:R")
+		(at 107.95 67.31 0)
+		(mirror y)
+		(unit 1)
+		(exclude_from_sim no)
+		(in_bom yes)
+		(on_board yes)
+		(dnp no)
+		(property "Reference" "R30"
+			(at 105.41 66.0399 0)
+			(effects
+				(font
+					(size 1.27 1.27)
+				)
+				(justify left)
+			)
+		)
+		(property "Value" "0"
+			(at 105.41 68.5799 0)
+			(effects
+				(font
+					(size 1.27 1.27)
+				)
+				(justify left)
+			)
+		)
+		(property "Footprint" "Resistor_SMD:R_0201_0603Metric"
+			(at 109.728 67.31 90)
+			(effects
+				(font
+					(size 1.27 1.27)
+				)
+				(hide yes)
+			)
+		)
+		(property "Datasheet" "~"
+			(at 107.95 67.31 0)
+			(effects
+				(font
+					(size 1.27 1.27)
+				)
+				(hide yes)
+			)
+		)
+		(property "Description" "Resistor"
+			(at 107.95 67.31 0)
+			(effects
+				(font
+					(size 1.27 1.27)
+				)
+				(hide yes)
+			)
+		)
+		(pin "2"
+		)
+		(pin "1"
+		)
+		(instances
+			(project "36mm PCB"
+				(path "/5882e07c-81e3-4e1e-9f7f-ac7d295520fe/658e32ce-0290-4965-9622-94e6b232efb2"
+					(reference "R30")
+					(unit 1)
+				)
