File: PCB/36mm PCB/Power.kicad_sch (KiCad schematic)
At the start: 20 parts, among them IC4 TPS22991BRAAR, IC5 MCP73831-2ACI_MC, J2 Conn_01x02_Socket, J3 Conn_01x02, Q7 2N7002KQBZ, SW5 SW_MEC_5E

Commit message: Modifs Mathieu
Parts:
- removed IC4: TPS22991BRAAR, SamacSys_Parts:TPS22991BRAAR, symbol SamacSys_Parts:TPS22991BRAAR
- added C1, C2: 1u, Capacitor_SMD:C_0402_1005Metric, symbol Device:C
- added R24, R25, R26, R27: 0, Resistor_SMD:R_0201_0603Metric, symbol Device:R_Small
Connections:
- net +3.3V: now also C2.1
- net +3V0: now also R16.1, C1.1; no longer SW5.2, SW5.4
- net Button press: now also R27.1; no longer R15.2, TPS3424A11C13ADRLR1.1 (PB)
- net GND: now also SW5.1, SW5.3, C1.2, C2.2; no longer R16.2
- net KeepOn: now also R24.2; no longer LDLN025PU1.3 (EN), TPS3424A11C13ADRLR1.6 (RESET/~RESET~)
- net Kill: now also R26.2; no longer TPS3424A11C13ADRLR1.8 (kill)
- net L-S press INT: now also R25.2; no longer TPS3424A11C13ADRLR1.7 (~INT~)
- new net: C20.2, R15.1, R16.2, SW5.2, SW5.4
- new net: R15.2, R27.2, TPS3424A11C13ADRLR1.1 (PB)
- new net: R25.1, TPS3424A11C13ADRLR1.7 (~INT~)
- new net: LDLN025PU1.3 (EN), R24.1, TPS3424A11C13ADRLR1.6 (RESET/~RESET~)
- new net: R26.1, TPS3424A11C13ADRLR1.8 (kill)
Other:
- moved on the sheet: R16, SW5

Commit message: STM32 BLE + H chip
Changed lines of the file:
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@@
 	)
 	(junction
+		(at 148.59 40.64)
+		(diameter 0)
+		(color 0 0 0 0)
+	)
+	(junction
 		(at 185.42 52.07)
 		(diameter 0)
@@
 	(wire
 		(pts
-			(xy 146.05 40.64) (xy 149.86 40.64)
+			(xy 146.05 40.64) (xy 148.59 40.64)
 		)
 		(stroke
@@
 	(wire
 		(pts
+			(xy 148.59 40.64) (xy 149.86 40.64)
+		)
+		(stroke
+			(width 0)
+			(type default)
+		)
+	)
+	(wire
+		(pts
 			(xy 121.92 81.28) (xy 125.73 81.28)
 		)
@@
 	(symbol
 		(lib_id "power:PWR_FLAG")
-		(at 146.05 40.64 0)
+		(at 148.59 40.64 0)
 		(unit 1)
 		(exclude_from_sim no)
@@
 		(dnp no)
 		(property "Reference" "#FLG01"
-			(at 146.05 38.735 0)
+			(at 148.59 38.735 0)
 			(effects
 				(font
@@
 		)
 		(property "Value" "PWR_FLAG"
-			(at 148.59 37.084 0)
+			(at 151.13 37.084 0)
 			(effects
 				(font
@@
 		)
 		(property "Footprint" ""
-			(at 146.05 40.64 0)
+			(at 148.59 40.64 0)
 			(effects
 				(font
@@
 		)
 		(property "Datasheet" "~"
-			(at 146.05 40.64 0)
+			(at 148.59 40.64 0)
 			(effects
 				(font
@@
 		)
 		(property "Description" "Special symbol for telling ERC where power comes from"
-			(at 146.05 40.64 0)
+			(at 148.59 40.64 0)
 			(effects
 				(font
